File: rpi5re/rpi5re.kicad_sch (KiCad schematic)
At the start: 24 parts, among them J1 USB_C_Receptacle, J13 HDMI_D_1.4, J16 UART, J2 HDMI_D_1.4, J2 Micro_SD_Card_Det1, J3 Conn_02x20_Odd_Even, J5 BAT, Q1 DMG7430LFGQ, SW1 SW_Push, U1 DA9091

Commit message: stuff
Parts:
- added J10: Bus_PCI_Express_x1, Connector_PCBEdge:BUS_PCIexpress_x1, symbol Connector:Bus_PCI_Express_x1
- added J10: ETHERNET, Connector_RJ:RJ45_UDE_RB1-125B8G1A, symbol Connector:RJ45_RB1-125B8G1A
- added J11: USB2, symbol Connector:USB_A_Stacked
- added J12: USB3, symbol Connector:USB3_A_Stacked
- added J14: PoE, symbol Connector_Generic:Conn_02x02_Odd_Even
- added J17: FAN, symbol Connector:Conn_01x04_Pin
- added J4: USB3_A_Stacked, symbol Connector:USB3_A_Stacked
- added J7: VID, symbol Connector:Conn_01x02_Socket
- added L1, L2, L3: 0.2uH, symbol Device:L
- added U2: RP2040, Package_DFN_QFN:QFN-56-1EP_7x7mm_P0.4mm_EP3.2x3.2mm, symbol MCU_RaspberryPi:RP2040
- J1: value USB_C_Receptacle -> PWR
- J13: value HDMI_D_1.4 -> HDMI11
- J2: value HDMI_D_1.4 -> HDMI10
- U1: value DA9091 -> Renesas DA9091
Connections:
- net at U1. (PGND): now also L3.2
- net at U1.24 (VBUCK3): now also L3.1
- net at U1.25 (VBUCK2): now also L2.1
- net at U1.26 (VBUCK1): now also L1.1
- net at U1.32 (VDD_BUCK1): now also L1.2
- new net: J10.A10 (+3.3V), J10.A9 (+3.3V), J10.B8 (+3.3V)
- new net: J10.A12 (GND), J10.A15 (GND), J10.A18 (GND), J10.A4 (GND), J10.B13 (GND), J10.B16 (GND), J10.B18 (GND), J10.B4 (GND), J10.B7 (GND)
- new net: J10.A2 (+12V), J10.A3 (+12V), J10.B1 (+12V), J10.B2 (+12V), J10.B3 (+12V)
- new net: U2.1 (IOVDD), U2.10 (IOVDD), U2.22 (IOVDD), U2.33 (IOVDD), U2.42 (IOVDD), U2.49 (IOVDD)
- new net: U2.23 (DVDD), U2.50 (DVDD)
- new net: L2.2, U1. (PGND)
- new net: J12.16 (DRAIN2), J12.19 (SHIELD)
